File: SplitKeyOne.kicad_pcb (KiCad board)
At the start: 2 copper layers, 121 parts, among them U1 MAX6951, U2 Teensy3.6_nopogo, U3 MAX6951

Commit message: Rough layout of right side.
Parts:
- added C7: C, Capacitors_SMD:C_0805_HandSoldering, F.Cu at (355.6, 31.8)
- added C8: 22uF, Capacitors_SMD:C_0805_HandSoldering, F.Cu at (355.6, 35.6)
- added C9: 0.1uF, Capacitors_SMD:C_0805_HandSoldering, F.Cu at (355.6, 26.7)
- added D100: D, Diodes_ThroughHole:D_DO-35_SOD27_P7.62mm_Horizontal, F.Cu at (415.3, 103.5)
- added D101: D, Diodes_ThroughHole:D_DO-35_SOD27_P7.62mm_Horizontal, F.Cu at (415.3, 122.6)
- added D102: D, Diodes_ThroughHole:D_DO-35_SOD27_P7.62mm_Horizontal, F.Cu at (415.3, 160.7)
- added D56: D, Diodes_ThroughHole:D_DO-35_SOD27_P7.62mm_Horizontal, F.Cu at (256.5, 59.1)
- added D57: D, Diodes_ThroughHole:D_DO-35_SOD27_P7.62mm_Horizontal, F.Cu at (256.5, 84.5)
- added D58: D, Diodes_ThroughHole:D_DO-35_SOD27_P7.62mm_Horizontal, F.Cu at (256.5, 103.5)
- added D59: D, Diodes_ThroughHole:D_DO-35_SOD27_P7.62mm_Horizontal, F.Cu at (256.5, 122.6)
- added D60: D, Diodes_ThroughHole:D_DO-35_SOD27_P7.62mm_Horizontal, F.Cu at (256.5, 141.6)
- added D61: D, Diodes_ThroughHole:D_DO-35_SOD27_P7.62mm_Horizontal, F.Cu at (256.5, 160.7)
- added D62: D, Diodes_ThroughHole:D_DO-35_SOD27_P7.62mm_Horizontal, F.Cu at (275.6, 59.1)
- added D63: D, Diodes_ThroughHole:D_DO-35_SOD27_P7.62mm_Horizontal, F.Cu at (275.6, 84.5)
- added D64: D, Diodes_ThroughHole:D_DO-35_SOD27_P7.62mm_Horizontal, F.Cu at (275.6, 103.5)
- added D65: D, Diodes_ThroughHole:D_DO-35_SOD27_P7.62mm_Horizontal, F.Cu at (275.6, 122.6)
- added D66: D, Diodes_ThroughHole:D_DO-35_SOD27_P7.62mm_Horizontal, F.Cu at (275.6, 141.6)
- added D67: D, Diodes_ThroughHole:D_DO-35_SOD27_P7.62mm_Horizontal, F.Cu at (294.6, 59.1)
- added D68: D, Diodes_ThroughHole:D_DO-35_SOD27_P7.62mm_Horizontal, F.Cu at (294.6, 84.5)
- added D69: D, Diodes_ThroughHole:D_DO-35_SOD27_P7.62mm_Horizontal, F.Cu at (294.6, 103.5)
- added D70: D, Diodes_ThroughHole:D_DO-35_SOD27_P7.62mm_Horizontal, F.Cu at (294.6, 122.6)
- added D71: D, Diodes_ThroughHole:D_DO-35_SOD27_P7.62mm_Horizontal, F.Cu at (294.6, 141.6)
- added D72: D, Diodes_ThroughHole:D_DO-35_SOD27_P7.62mm_Horizontal, F.Cu at (294.6, 160.7)
- added D73: D, Diodes_ThroughHole:D_DO-35_SOD27_P7.62mm_Horizontal, F.Cu at (313.7, 160.7)
- added D74: D, Diodes_ThroughHole:D_DO-35_SOD27_P7.62mm_Horizontal, F.Cu at (313.7, 59.1)
- added D75: D, Diodes_ThroughHole:D_DO-35_SOD27_P7.62mm_Horizontal, F.Cu at (313.7, 84.5)
- added D76: D, Diodes_ThroughHole:D_DO-35_SOD27_P7.62mm_Horizontal, F.Cu at (313.7, 103.5)
- added D77: D, Diodes_ThroughHole:D_DO-35_SOD27_P7.62mm_Horizontal, F.Cu at (313.7, 122.6)
- added D78: D, Diodes_ThroughHole:D_DO-35_SOD27_P7.62mm_Horizontal, F.Cu at (313.7, 141.6)
- added D79: D, Diodes_ThroughHole:D_DO-35_SOD27_P7.62mm_Horizontal, F.Cu at (332.7, 59.1)
- added D80: D, Diodes_ThroughHole:D_DO-35_SOD27_P7.62mm_Horizontal, F.Cu at (332.7, 84.5)
- added D81: D, Diodes_ThroughHole:D_DO-35_SOD27_P7.62mm_Horizontal, F.Cu at (332.7, 103.5)
- added D82: D, Diodes_ThroughHole:D_DO-35_SOD27_P7.62mm_Horizontal, F.Cu at (332.7, 122.6)
- added D83: D, Diodes_ThroughHole:D_DO-35_SOD27_P7.62mm_Horizontal, F.Cu at (332.7, 141.6)
- added D84: D, Diodes_ThroughHole:D_DO-35_SOD27_P7.62mm_Horizontal, F.Cu at (332.7, 160.7)
- added D85: D, Diodes_ThroughHole:D_DO-35_SOD27_P7.62mm_Horizontal, F.Cu at (351.8, 59.1)
- added D86: D, Diodes_ThroughHole:D_DO-35_SOD27_P7.62mm_Horizontal, F.Cu at (351.8, 84.5)
- added D87: D, Diodes_ThroughHole:D_DO-35_SOD27_P7.62mm_Horizontal, F.Cu at (351.8, 103.5)
- added D88: D, Diodes_ThroughHole:D_DO-35_SOD27_P7.62mm_Horizontal, F.Cu at (351.8, 122.6)
- added D89: D, Diodes_ThroughHole:D_DO-35_SOD27_P7.62mm_Horizontal, F.Cu at (351.8, 141.6)
- added D90: D, Diodes_ThroughHole:D_DO-35_SOD27_P7.62mm_Horizontal, F.Cu at (370.8, 59.1)
- added D91: D, Diodes_ThroughHole:D_DO-35_SOD27_P7.62mm_Horizontal, F.Cu at (370.8, 103.5)
- added D92: D, Diodes_ThroughHole:D_DO-35_SOD27_P7.62mm_Horizontal, F.Cu at (370.8, 160.7)
- added D93: D, Diodes_ThroughHole:D_DO-35_SOD27_P7.62mm_Horizontal, F.Cu at (389.9, 59.1)
- added D94: D, Diodes_ThroughHole:D_DO-35_SOD27_P7.62mm_Horizontal, F.Cu at (380.4, 84.5)
- added D95: D, Diodes_ThroughHole:D_DO-35_SOD27_P7.62mm_Horizontal, F.Cu at (389.9, 103.5)
- added D96: D, Diodes_ThroughHole:D_DO-35_SOD27_P7.62mm_Horizontal, F.Cu at (389.9, 122.6)
- added D97: D, Diodes_ThroughHole:D_DO-35_SOD27_P7.62mm_Horizontal, F.Cu at (389.9, 160.7)
- added D98: D, Diodes_ThroughHole:D_DO-35_SOD27_P7.62mm_Horizontal, F.Cu at (415.3, 59.1)
- added D99: D, Diodes_ThroughHole:D_DO-35_SOD27_P7.62mm_Horizontal, F.Cu at (415.3, 84.5)
- added R3: 56k, Resistors_SMD:R_0805_HandSoldering, F.Cu at (342.3, 40.0)
- added S100: RESC, Custom:CHERRY-MX-LED-Socket, F.Cu at (425.4, 63.5)
- added S101: U8, Custom:CHERRY-MX-LED-Socket, F.Cu at (425.4, 88.9)
- added S102: U10, Custom:CHERRY-MX-LED-Socket, F.Cu at (425.4, 108.0)
- added S56: U6, Custom:CHERRY-MX-LED-Socket, F.Cu at (266.7, 63.5)
- added S57: NUM7, Custom:CHERRY-MX-LED-Socket, F.Cu at (266.7, 88.9)
- added S58: y, Custom:CHERRY-MX-LED-Socket, F.Cu at (257.2, 108.0)
- added S59: h, Custom:CHERRY-MX-LED-Socket, F.Cu at (261.9, 127.0)
- added S60: n, Custom:CHERRY-MX-LED-Socket, F.Cu at (271.5, 146.1)
- added S61: RSPACE, Custom:CHERRY-MX-LED-Socket, F.Cu at (266.7, 165.1)
- added S62: F6, Custom:CHERRY-MX-LED-Socket, F.Cu at (285.8, 63.5)
- added S63: NUM8, Custom:CHERRY-MX-LED-Socket, F.Cu at (285.8, 88.9)
- added S64: u, Custom:CHERRY-MX-LED-Socket, F.Cu at (276.2, 108.0)
- added S65: j, Custom:CHERRY-MX-LED-Socket, F.Cu at (281.0, 127.0)
- added S66: m, Custom:CHERRY-MX-LED-Socket, F.Cu at (290.5, 146.1)
- added S67: F7, Custom:CHERRY-MX-LED-Socket, F.Cu at (304.8, 63.5)
- added S68: NUM9, Custom:CHERRY-MX-LED-Socket, F.Cu at (304.8, 88.9)
- added S69: i, Custom:CHERRY-MX-LED-Socket, F.Cu at (295.3, 108.0)
- added S70: k, Custom:CHERRY-MX-LED-Socket, F.Cu at (300.0, 127.0)
- added S71: COMMA, Custom:CHERRY-MX-LED-Socket, F.Cu at (309.6, 146.1)
- added S72: U14, Custom:CHERRY-MX-LED-Socket, F.Cu at (301.6, 165.1)
- added S73: U15, Custom:CHERRY-MX-LED-Socket, F.Cu at (328.6, 165.1)
- added S74: F8, Custom:CHERRY-MX-LED-Socket, F.Cu at (323.9, 63.5)
- added S75: NUM0, Custom:CHERRY-MX-LED-Socket, F.Cu at (323.9, 88.9)
- added S76: o, Custom:CHERRY-MX-LED-Socket, F.Cu at (314.3, 108.0)
- added S77: l, Custom:CHERRY-MX-LED-Socket, F.Cu at (319.1, 127.0)
- added S78: PERIOD, Custom:CHERRY-MX-LED-Socket, F.Cu at (328.6, 146.1)
- added S79: F9, Custom:CHERRY-MX-LED-Socket, F.Cu at (342.9, 63.5)
- added S80: MINUS, Custom:CHERRY-MX-LED-Socket, F.Cu at (342.9, 88.9)
- added S81: p, Custom:CHERRY-MX-LED-Socket, F.Cu at (333.4, 108.0)
- added S82: colon, Custom:CHERRY-MX-LED-Socket, F.Cu at (338.1, 127.0)
- added S83: SLASH, Custom:CHERRY-MX-LED-Socket, F.Cu at (347.7, 146.1)
- added S84: RALT, Custom:CHERRY-MX-LED-Socket, F.Cu at (357.2, 165.1)
- added S85: F10, Custom:CHERRY-MX-LED-Socket, F.Cu at (361.9, 63.5)
- added S86: EQUALS, Custom:CHERRY-MX-LED-Socket, F.Cu at (361.9, 88.9)
- added S87: {, Custom:CHERRY-MX-LED-Socket, F.Cu at (352.4, 108.0)
- added S88: quote, Custom:CHERRY-MX-LED-Socket, F.Cu at (357.2, 127.0)
- added S89: RSHIFT, Custom:CHERRY-MX-LED-Socket, F.Cu at (381.0, 146.1)
- added S90: F11, Custom:CHERRY-MX-LED-Socket, F.Cu at (381.0, 63.5)
- added S91: ], Custom:CHERRY-MX-LED-Socket, F.Cu at (371.5, 108.0)
- added S92: RWIN, Custom:CHERRY-MX-LED-Socket, F.Cu at (377.8, 165.1)
- added S93: F12, Custom:CHERRY-MX-LED-Socket, F.Cu at (400.1, 63.5)
- added S94: BACKSPACE, Custom:CHERRY-MX-LED-Socket, F.Cu at (390.5, 88.9)
- added S95: BACKSLASH, Custom:CHERRY-MX-LED-Socket, F.Cu at (395.3, 108.0)
- added S96: ENTER, Custom:CHERRY-MX-LED-Socket, F.Cu at (388.1, 127.0)
- added S97: RCTRL, Custom:CHERRY-MX-LED-Socket, F.Cu at (398.5, 165.1)
- added S98: U12, Custom:CHERRY-MX-LED-Socket, F.Cu at (425.4, 127.0)
- added S99: RENTER, Custom:CHERRY-MX-LED-Socket, F.Cu at (425.4, 155.6)
- added U4: MAX6951, Housings_SSOP:TSSOP-16-1EP_4.4x5mm_Pitch0.65mm, F.Cu at (349.2, 38.1)
- S14: value ESC -> LESC
Connections:
- U2 pad 24: (no net) -> C12
- U2 pad 30: (no net) -> C13
- U2 pad 31: (no net) -> C14
- U2 pad 32: (no net) -> C15
- U2 pad 33: (no net) -> C16
- U2 pad 34: (no net) -> C17
- U2 pad 35: (no net) -> C18
- U2 pad 36: (no net) -> C19
- U2 pad 41: (no net) -> C20
- U2 pad 48: (no net) -> LED_CS3

Commit message: Hopefully final layout of keys.
Parts:
- moved S84 7.14 mm to (350.0, 165.1)
- moved S72 6.35 mm to (295.3, 165.1)
- moved S73 4.76 mm to (323.9, 165.1)
- moved S92 3.97 mm to (373.9, 165.1)
- moved S71 2.38 mm to (307.2, 146.1)
- moved S78 2.38 mm to (326.2, 146.1)
- moved S83 2.38 mm to (345.3, 146.1)
- moved S60 2.38 mm to (269.1, 146.1)
- moved S61 2.38 mm to (264.3, 165.1)
- moved S66 2.38 mm to (288.1, 146.1)
- moved S97 0.79 mm to (397.7, 165.1)
Changed lines of the file:
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@@
     (area 18.555 23.2846 433.524001 173.301001)
     (thickness 1.6)
-    (drawings 1)
+    (drawings 2)
     (tracks 937)
     (zones 0)
@@
     (visible_elements 7FFFFFFF)
     (pcbplotparams
-      (layerselection 0x00f30_00000000)
+      (layerselection 0x00020_00000000)
       (usegerberextensions false)
       (excludeedgelayer true)
@@
   )
   (module Custom:CHERRY-MX-LED-Socket (layer F.Cu)
-    (at 271.4625 146.05)
+    (at 269.08125 146.05)
     (attr virtual)
     (fp_text reference S60 (at -4.572 5.334) (layer F.SilkS)
@@
   )
   (module Custom:CHERRY-MX-LED-Socket (layer F.Cu)
-    (at 266.7 165.1)
+    (at 264.31875 165.1)
     (attr virtual)
     (fp_text reference S61 (at -4.572 5.334) (layer F.SilkS)
@@
   )
   (module Custom:CHERRY-MX-LED-Socket (layer F.Cu)
-    (at 290.5125 146.05)
+    (at 288.13125 146.05)
     (attr virtual)
     (fp_text reference S66 (at -4.572 5.334) (layer F.SilkS)
@@
   )
   (module Custom:CHERRY-MX-LED-Socket (layer F.Cu)
-    (at 309.5625 146.05)
+    (at 307.18125 146.05)
     (attr virtual)
     (fp_text reference S71 (at -4.572 5.334) (layer F.SilkS)
@@
   )
   (module Custom:CHERRY-MX-LED-Socket (layer F.Cu)
-    (at 301.625 165.1)
+    (at 295.275 165.1)
     (attr virtual)
     (fp_text reference S72 (at -4.572 5.334) (layer F.SilkS)
@@
   )
   (module Custom:CHERRY-MX-LED-Socket (layer F.Cu)
-    (at 328.6125 165.1)
+    (at 323.85 165.1)
     (attr virtual)
     (fp_text reference S73 (at -4.572 5.334) (layer F.SilkS)
@@
   )
   (module Custom:CHERRY-MX-LED-Socket (layer F.Cu)
-    (at 328.6125 146.05)
+    (at 326.23125 146.05)
     (attr virtual)
     (fp_text reference S78 (at -4.572 5.334) (layer F.SilkS)
@@
   )
   (module Custom:CHERRY-MX-LED-Socket (layer F.Cu)
-    (at 347.6625 146.05)
+    (at 345.28125 146.05)
     (attr virtual)
     (fp_text reference S83 (at -4.572 5.334) (layer F.SilkS)
@@
   )
   (module Custom:CHERRY-MX-LED-Socket (layer F.Cu)
-    (at 357.1875 165.1)
+    (at 350.04375 165.1)
     (attr virtual)
     (fp_text reference S84 (at -4.572 5.334) (layer F.SilkS)
@@
   )
   (module Custom:CHERRY-MX-LED-Socket (layer F.Cu)
-    (at 377.825 165.1)
+    (at 373.85625 165.1)
     (attr virtual)
     (fp_text reference S92 (at -4.572 5.334) (layer F.SilkS)
@@
   )
   (module Custom:CHERRY-MX-LED-Socket (layer F.Cu)
-    (at 398.4625 165.1)
+    (at 397.66875 165.1)
     (attr virtual)
     (fp_text reference S97 (at -4.572 5.334) (layer F.SilkS)
@@
     )
   )
+  (gr_line (start 409.575 164.2745) (end 409.575 167.767) (angle 90) (layer Dwgs.User) (width 0.2))
   (gr_line (start 234.0864 55.7784) (end 234.0864 56.1594) (angle 90) (layer Dwgs.User) (width 0.2))
   (segment (start 246.3238 29.0322) (end 246.3746 29.083) (width 0.25) (layer B.Cu) (net 1))

Commit message: Final key placement.
Parts:
- moved S71 2.38 mm to (309.6, 146.1)
- moved S78 2.38 mm to (328.6, 146.1)
- moved S83 2.38 mm to (347.7, 146.1)
- moved S89 2.38 mm to (383.4, 146.1)
- moved S60 2.38 mm to (271.5, 146.1)
- moved S66 2.38 mm to (290.5, 146.1)
Changed lines of the file:
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@@
   )
   (module Custom:CHERRY-MX-LED-Socket (layer F.Cu)
-    (at 269.08125 146.05)
+    (at 271.4625 146.05)
     (attr virtual)
     (fp_text reference S60 (at -4.572 5.334) (layer F.SilkS)
@@
   )
   (module Custom:CHERRY-MX-LED-Socket (layer F.Cu)
-    (at 288.13125 146.05)
+    (at 290.5125 146.05)
     (attr virtual)
     (fp_text reference S66 (at -4.572 5.334) (layer F.SilkS)
@@
   )
   (module Custom:CHERRY-MX-LED-Socket (layer F.Cu)
-    (at 307.18125 146.05)
+    (at 309.5625 146.05)
     (attr virtual)
     (fp_text reference S71 (at -4.572 5.334) (layer F.SilkS)
@@
   )
   (module Custom:CHERRY-MX-LED-Socket (layer F.Cu)
-    (at 326.23125 146.05)
+    (at 328.6125 146.05)
     (attr virtual)
     (fp_text reference S78 (at -4.572 5.334) (layer F.SilkS)
@@
   )
   (module Custom:CHERRY-MX-LED-Socket (layer F.Cu)
-    (at 345.28125 146.05)
+    (at 347.6625 146.05)
     (attr virtual)
     (fp_text reference S83 (at -4.572 5.334) (layer F.SilkS)
@@
   )
   (module Custom:CHERRY-MX-LED-Socket (layer F.Cu)
-    (at 381 146.05)
+    (at 383.38125 146.05)
     (attr virtual)
     (fp_text reference S89 (at -4.572 5.334) (layer F.SilkS)

Commit message: More routing.
Parts:
- S18, S20, S55, S89, S94, S96, S99: footprint Custom:CHERRY-MX-LED-Socket -> SplitKeyOne:CHERRY-MX-LED-Socket-2-stabilizer
- moved D99 66.7 mm to (415.3, 151.1)
- moved D98 63.4 mm to (415.3, 122.4)
- moved D102 57.0 mm to (415.3, 103.6)
- moved D100 44.4 mm to (415.3, 59.1)
- moved D101 38.1 mm to (415.2, 84.5)
- moved D89 21.1 mm to (372.9, 141.7)
- moved D96 12.1 mm to (377.8, 122.6)
- moved D72 9.65 mm to (285.0, 160.5)
- moved D58 9.53 mm to (247.0, 103.5)
- moved D81 9.53 mm to (323.2, 103.5)
- moved D87 9.53 mm to (342.3, 103.5)
- moved D64 9.52 mm to (266.1, 103.5)
- moved D69 9.52 mm to (285.1, 103.5)
- moved D76 9.52 mm to (304.2, 103.5)
- moved D91 9.52 mm to (361.3, 103.5)
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Connections:
- U1 pad 17: GND -> (no net)
- U3 pad 17: GND -> (no net)
- U4 pad 17: GND -> (no net)
Routing:
- net R6: track 207.3 -> 369.5 mm
- net /right/LED5: track 0.00 -> 147.1 mm
- net C15: track 0.00 -> 21.3 mm
- net C14: track 0.00 -> 21.3 mm
- net C12: track 0.00 -> 21.3 mm
- net C20: track 0.00 -> 17.8 mm
- net C19: track 0.00 -> 17.8 mm
- net C17: track 0.00 -> 17.8 mm
- net C16: track 0.00 -> 17.8 mm
- net C13: track 0.00 -> 17.7 mm
- net C18: track 0.00 -> 14.2 mm
- net Net-(D97-Pad1): track 0.00 -> 7.60 mm
- net Net-(D59-Pad1): track 0.00 -> 7.51 mm
- net Net-(D60-Pad1): track 0.00 -> 7.49 mm
- net Net-(D95-Pad1): track 0.00 -> 7.46 mm
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
Commit message: More routing.
Parts:
- moved D82 0.25 mm to (328.2, 122.7)
Routing:
- net R4: track 135.3 -> 394.0 mm
- net R5: track 146.8 -> 360.5 mm
- net R1: track 203.2 -> 393.7 mm
- net R3: track 203.3 -> 393.8 mm
- net R2: track 203.3 -> 393.6 mm
- net /right/LED3: track 0.00 -> 182.7 mm
- net /right/LED1: track 0.00 -> 176.2 mm
- net /right/LED2: track 0.00 -> 164.0 mm
- net /right/LED0: track 0.00 -> 154.2 mm
- net C14: track 21.3 -> 159.9 mm
- net C12: track 21.3 -> 152.0 mm
- net C18: track 14.2 -> 143.3 mm
- net C15: track 21.3 -> 149.6 mm
- net C19: track 17.8 -> 143.7 mm
- net /right/LED4: track 0.00 -> 125.4 mm
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
Commit message: Board routed.
Parts:
- C4, C5, C6, C7, C8, C9, R2, R3, U3, U4: moved to B.Cu
- U2: value Teensy3.6_nopogo -> Teensy3.6
- moved U2 29.3 mm to (185.5, 33.4), turned to 0 degrees
- moved C9 23.7 mm to (343.5, 47.1), turned to 270 degrees
- moved C3 22.9 mm to (253.9, 48.0), turned to 270 degrees
- moved C2 19.3 mm to (251.6, 48.0), turned to 270 degrees
- moved C1 16.9 mm to (262.4, 47.9)
- moved C7 15.3 mm to (353.8, 47.0), turned to 270 degrees
- moved C8 15.2 mm to (345.7, 47.1), turned to 270 degrees
- moved R1 11.4 mm to (260.5, 37.2), turned to 90 degrees
- moved R3 10.6 mm to (352.2, 36.3), turned to 90 degrees
- moved C4 9.88 mm to (131.3, 47.6), turned to 270 degrees
- moved C6 7.27 mm to (120.5, 47.5), turned to 270 degrees
- moved R2 5.74 mm to (129.3, 36.7), turned to 90 degrees
- moved U4 4.60 mm to (349.8, 42.7), turned to 270 degrees
- moved C5 4.38 mm to (122.7, 47.5), turned to 270 degrees
- moved U1 3.31 mm to (258.2, 43.6), turned to 270 degrees
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Connections:
- C1 pad 1: (no net) -> Net-(C1-Pad1)
- U1 pad 17: (no net) -> GND
- U1 pad 9: (no net) -> Net-(C1-Pad1)
- U2 pad 30: C13 -> C20
- U2 pad 31: C14 -> C19
- U2 pad 32: C15 -> C18
- U2 pad 33: C16 -> C17
- U2 pad 34: C17 -> C16
- U2 pad 35: C18 -> C15
- U2 pad 36: C19 -> C14
- U2 pad 41: C20 -> C13
- U3 pad 17: (no net) -> GND
- U4 pad 17: (no net) -> GND
Routing:
- net /right/LED5: track 147.1 -> 488.6 mm, vias 0 -> 3
- net SCK: track 0.00 -> 330.7 mm, vias 0 -> 4
- net /right/LED6: track 0.00 -> 303.1 mm, vias 0 -> 2
- net /right/LED2: track 164.0 -> 458.0 mm, vias 0 -> 3
- net /right/LED1: track 176.2 -> 457.3 mm, vias 0 -> 5
- net /right/LED3: track 182.7 -> 446.2 mm, vias 0 -> 5
- net /right/LED0: track 154.2 -> 413.0 mm, vias 0 -> 4
- net /right/LED4: track 125.4 -> 382.9 mm, vias 0 -> 4
- net C20: track 128.6 -> 373.4 mm
- net MOSI: track 0.00 -> 238.8 mm, vias 0 -> 5
- net /right/LED8: track 0.00 -> 238.0 mm, vias 0 -> 2
- net C19: track 143.7 -> 364.7 mm
- net /right/LED7: track 0.00 -> 214.2 mm, vias 0 -> 2
- net C18: track 143.3 -> 347.5 mm
- net LED_CS3: track 0.00 -> 190.0 mm, vias 0 -> 1
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- added copper zone on F.Cu, net 5V
- added copper zone on B.Cu, net GND
Other:
- board outline added: 426.2 x 156.7 mm

Commit message: Mounting holes.
Parts:
- added J1: M04, Custom:SparkFun-1X04_LOCK, F.Cu at (179.2, 22.1)
- added J2: M04, Custom:SparkFun-1X04_LOCK, F.Cu at (182.8, 22.1)
- added REF**: MountingHole_3.2mm_M3, Mounting_Holes:MountingHole_3.2mm_M3, F.Cu at (408.6, 107.3)
- added REF**: MountingHole_3.2mm_M3, Mounting_Holes:MountingHole_3.2mm_M3, F.Cu at (438.3, 23.1)
- added REF**: MountingHole_3.2mm_M3, Mounting_Holes:MountingHole_3.2mm_M3, F.Cu at (19.2, 23.2)
- added REF**: MountingHole_3.2mm_M3, Mounting_Holes:MountingHole_3.2mm_M3, F.Cu at (44.9, 107.5)
- added REF**: MountingHole_3.2mm_M3, Mounting_Holes:MountingHole_3.2mm_M3, F.Cu at (266.6, 75.9)
- added REF**: MountingHole_3.2mm_M3, Mounting_Holes:MountingHole_3.2mm_M3, F.Cu at (216.1, 124.8)
- added REF**: MountingHole_3.2mm_M3, Mounting_Holes:MountingHole_3.2mm_M3, F.Cu at (171.3, 76.3)
- added REF**: MountingHole_3.2mm_M3, Mounting_Holes:MountingHole_3.2mm_M3, F.Cu at (249.6, 172.7)
- added REF**: MountingHole_3.2mm_M3, Mounting_Holes:MountingHole_3.2mm_M3, F.Cu at (185.2, 172.7)
- added REF**: MountingHole_3.2mm_M3, Mounting_Holes:MountingHole_3.2mm_M3, F.Cu at (19.2, 172.7)
- added REF**: MountingHole_3.2mm_M3, Mounting_Holes:MountingHole_3.2mm_M3, F.Cu at (438.3, 172.7)
- U2: value Teensy3.6 -> Teensy3.6_nopogo
Connections:
- U2 pad 42: (no net) -> /G15
- U2 pad 43: (no net) -> /G16
- U2 pad 45: (no net) -> SDA
- U2 pad 46: (no net) -> SCL
Routing:
- net GND: track 0.00 -> 61.1 mm
- net /G16: track 0.00 -> 6.36 mm
- net /G15: track 0.00 -> 6.28 mm
- net SDA: track 0.00 -> 5.33 mm
- net /LED1: track 269.5 -> 274.3 mm
- net SCL: track 0.00 -> 4.24 mm
- net /right/LED0: track 413.0 -> 415.9 mm

Commit message: Making outlines for routing the plate.
Parts:
- S5: footprint Custom:CHERRY-MX-LED-Socket -> SplitKeyOne:CHERRY-MX-LED-Socket
